File: r60-std.kicad_pcb (KiCad board)
At the start: 2 copper layers, 285.8 x 95.3 mm, 153 parts, among them K0 ESC, K0A1 0, K0B1 MINUS, K0C1 EQUAL, K0D1 BACKSP, K1 1, K10 TAB, K11 Q, K12 W, K13 E, K14 R, K15 T, K16 Y, K17 U, K18 I, K19 O, K1A1 P, K1B1 LBRACE, K1C1 RBRACE, K1D1 BS_PIPE, K2 2, K20 CAPS, K20-S1 CAPS, K21 A, K22 S, K23 D, K24 F, K25 G, K26 H, K27 J, K28 K, K29 L, K2A1 COLON, K2B1 QUOTE, K2C1 ISOHASH, K2D1 ENTER, K2D2 ISOENTER, K3 3, K30 LSHIFT, K30-I1 ISOLSHIFT, K31 ISOPIPE, K32 Z, K33 X, K34 C, K35 V, K36 B, K37 N, K38 M, K39 COMMA, K3A1 DOT, K3B1 SLASH, K3C1 RSHIFT, K4 4, K40 LCTL, K41 LWIN, K42 LALT, K45 SPACE, K48 RALT, K49 RWIN, K4A1 RGUI, K4B1 RCTL, K5 5, K6 6, K7 7, K8 8, K9 9, P1 USB_B, P2 SPKR, SW1 SW_Push, U1 ATmega32U4-AU, Y1 16MHz

Commit message: First pass at r4 design
Remove ISO layouts, keep stepped capslock/ctrl.  Allow for
either 6.25u space or 1.25/2.25/2.75 split space. Move to
0603 footprints near atmega to handle smaller space due to
split spacebar.  Switch atmega from -AU in 44 TQFP to -MU
part in 44 QFN, again to deal with less room due to split
spacebar.
Parts:
- removed D2C1, D3C1: D, Keyboard:D_0805
- removed G***: LOGO, logos:ron-test
- removed K2C1: ISOHASH, Keyboard:CHERRY_PCB_100H
- removed K2D2: ISOENTER, Keyboard:CHERRY_PCB_200H
- removed K30-I1: ISOLSHIFT, Keyboard:CHERRY_PCB_125H
- removed K3C1: RSHIFT, Keyboard:CHERRY_PCB_275H
- removed P2: SPKR, Pin_Headers:Pin_Header_Straight_1x02_Pitch2.54mm
- added D43: D, Keyboard:D_0805, B.Cu at (113.3, 135.7)
- added D44: D, Keyboard:D_0805, B.Cu at (146.4, 135.7)
- added K43: LFN, Keyboard:CHERRY_PCB_125H, F.Cu at (111.9, 128.6)
- added K44: SSPACE-1, Keyboard:CHERRY_PCB_225H, F.Cu at (145.3, 128.6)
- added K45-1: SSPACE-2, Keyboard:CHERRY_PCB_275H, F.Cu at (192.9, 128.6)
- added LS1: AST1109MLT, Keyboard:AST1109ML-SMT, B.Cu at (185.7, 104.8)
- added REF**: Via-Stitch, Keyboard:Via-Stitch, F.Cu at (34.4, 94.2)
- added REF**: Via-Stitch, Keyboard:Via-Stitch, F.Cu at (306.6, 122.9)
- added REF**: Via-Stitch, Keyboard:Via-Stitch, F.Cu at (127.8, 120.0)
- added REF**: Via-Stitch, Keyboard:Via-Stitch, F.Cu at (155.8, 126.8)
- added REF**: Via-Stitch, Keyboard:Via-Stitch, F.Cu at (162.3, 118.2)
- added REF**: Via-Stitch, Keyboard:Via-Stitch, F.Cu at (173.4, 118.2)
- added REF**: Via-Stitch, Keyboard:Via-Stitch, F.Cu at (139.2, 133.6)
- added REF**: Via-Stitch, Keyboard:Via-Stitch, F.Cu at (125.7, 129.6)
- added REF**: Via-Stitch, Keyboard:Via-Stitch, F.Cu at (101.2, 132.2)
- added REF**: Via-Stitch, Keyboard:Via-Stitch, F.Cu at (73.8, 134.4)
- added REF**: Via-Stitch, Keyboard:Via-Stitch, F.Cu at (34.9, 47.3)
- added REF**: Via-Stitch, Keyboard:Via-Stitch, F.Cu at (85.6, 123.5)
- added REF**: Via-Stitch, Keyboard:Via-Stitch, F.Cu at (58.5, 47.9)
- added REF**: Via-Stitch, Keyboard:Via-Stitch, F.Cu at (109.8, 49.2)
- added REF**: Via-Stitch, Keyboard:Via-Stitch, F.Cu at (117.5, 87.1)
- added REF**: Via-Stitch, Keyboard:Via-Stitch, F.Cu at (196.1, 85.9)
- added REF**: Via-Stitch, Keyboard:Via-Stitch, F.Cu at (200.0, 52.8)
- added REF**: Via-Stitch, Keyboard:Via-Stitch, F.Cu at (306.5, 53.0)
- added REF**: Via-Stitch, Keyboard:Via-Stitch, F.Cu at (306.5, 89.2)
- C1, C2, C3, C4, C5, C6, C7, C8: footprint Capacitors_SMD:C_0805 -> Capacitors_SMD:C_0603
- K0D1: footprint Keyboard:CHERRY_PCB_200H -> Keyboard:CHERRY_PCB_200H_INVERTED
- K31: value ISOPIPE -> Z
- K32: value Z -> x
- K33: value X -> C
- K34: value C -> V
- K35: value V -> B
- K36: value B -> N
- K37: value N -> M
- K38: value M -> COMMA
- K39: value COMMA -> DOT
- K3A1: value DOT -> SLASH
- K3B1: value SLASH -> RSHIFT; footprint Keyboard:CHERRY_PCB_100H -> Keyboard:CHERRY_PCB_275H
- R4: footprint Keyboard:RC_0805 -> Resistors_SMD:R_0603
- U1: footprint Housings_QFP:TQFP-44_10x10mm_Pitch0.8mm -> Housings_DFN_QFN:QFN-44-1EP_7x7mm_Pitch0.5mm
- moved R5 60.0 mm to (184.4, 114.6)
- moved C9 59.9 mm to (187.1, 114.6)
- moved Y1 49.7 mm to (167.6, 128.6)
- moved C1 49.5 mm to (167.6, 125.5)
- moved C2 49.4 mm to (167.5, 131.7)
- moved C6 47.4 mm to (167.5, 133.1)
- moved C5 45.2 mm to (172.1, 122.8), turned to 180 degrees
- moved U1 43.8 mm to (175.7, 127.8)
- moved R4 39.1 mm to (182.7, 123.3)
- moved C3 39.0 mm to (182.0, 131.1)
- moved C4 38.5 mm to (181.9, 124.8)
- moved D3B1 35.9 mm to (289.3, 115.5)
- moved K3B1 35.7 mm to (288.1, 109.5)
- moved C7 33.9 mm to (177.4, 133.9), turned to 270 degrees
- moved C8 30.8 mm to (174.4, 133.9), turned to 270 degrees
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Routing:
- net Net-(R5-Pad1): track 157.7 -> 14.0 mm
- net /C13: track 254.5 -> 186.9 mm
- net /C1: track 152.4 -> 211.9 mm, vias 0 -> 3
- net Net-(R3-Pad2): track 101.8 -> 160.1 mm
- net /R1: track 327.1 -> 384.3 mm
- net /C2: track 127.5 -> 183.3 mm, vias 1 -> 2
- net /C3: track 97.0 -> 150.3 mm
- net Net-(R1-Pad2): track 148.7 -> 201.6 mm
- net Net-(R2-Pad1): track 153.0 -> 205.4 mm
- net /C8: track 191.3 -> 140.5 mm
- net /C10: track 237.5 -> 188.4 mm
- net /R0: track 355.1 -> 401.9 mm
- net /R2: track 311.9 -> 357.8 mm
- net VCC: track 211.2 -> 255.5 mm, vias 0 -> 3
- net /C0: track 191.0 -> 234.0 mm, vias 0 -> 2
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Other:
- board text added: "R60 Standard Board Rev 4.0"
- board text added: "github.com/rpedde/r60-std r4.0"
- board text removed: "R60 Standard Board Rev 3.0"
- board text removed: "github.com/rpedde/r60-std"
